File: KiCAD/anemometer_board/anemometer_board.kicad_pcb (KiCad board)
At the start: 2 copper layers, 66 x 66 mm, 12 parts, among them J1 SOLAR, J2 BATT, U1 TCRT5000, U2 TC4056A_BREAKOUT, U3 LM393, U4 REGULATOR

Commit message: Fix IR connections on PCB. Deploy as PCB V1.1
Parts:
- moved R1 5.08 mm to (76.2, 83.8)
- moved R2 5.08 mm to (81.3, 83.8)
Connections:
- U1 pad 2: Net-(R1-Pad2) -> Net-(R2-Pad2)
- U1 pad 4: Net-(R2-Pad2) -> Net-(R1-Pad2)
Routing:
- net Net-(R2-Pad2): track 26.2 -> 21.2 mm
Other:
- board text added: "ANEMOMETER BOARD V1.1"
- board text removed: "ANEMOMETER BOARD V1.0"
Changed lines of the file:
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@@
   )
   (module Resistor_THT:R_Axial_DIN0204_L3.6mm_D1.6mm_P7.62mm_Horizontal (layer B.Cu)
-    (at 76.2 83.82 270)
+    (at 81.28 83.82 270)
     (descr "Resistor, Axial_DIN0204 series, Axial, Horizontal, pin pitch=7.62mm, 0.167W, length*diameter=3.6*1.6mm^2, http://cdn-reichelt.de/documents/datenblatt/B400/1_4W%23YAG.pdf")
     (tags "Resistor Axial_DIN0204 series Axial Horizontal pin pitch 7.62mm 0.167W length 3.6mm diameter 1.6mm")
@@
   )
   (module Resistor_THT:R_Axial_DIN0204_L3.6mm_D1.6mm_P7.62mm_Horizontal (layer B.Cu)
-    (at 81.28 83.82 270)
+    (at 76.2 83.82 270)
     (descr "Resistor, Axial_DIN0204 series, Axial, Horizontal, pin pitch=7.62mm, 0.167W, length*diameter=3.6*1.6mm^2, http://cdn-reichelt.de/documents/datenblatt/B400/1_4W%23YAG.pdf")
     (tags "Resistor Axial_DIN0204 series Axial Horizontal pin pitch 7.62mm 0.167W length 3.6mm diameter 1.6mm")
@@
     )
     (pad 4 thru_hole circle (at 3.81 0 180) (size 2 2) (drill 0.8) (layers *.Cu *.Mask)
+      (net 34 "Net-(R1-Pad2)"))
+    (pad 3 thru_hole circle (at 1.27 0 180) (size 2 2) (drill 0.8) (layers *.Cu *.Mask)
+      (net 2 GND))
+    (pad 2 thru_hole circle (at -1.27 0 180) (size 2 2) (drill 0.8) (layers *.Cu *.Mask)
       (net 35 "Net-(R2-Pad2)"))
-    (pad 3 thru_hole circle (at 1.27 0 180) (size 2 2) (drill 0.8) (layers *.Cu *.Mask)
-      (net 2 GND))
-    (pad 2 thru_hole circle (at -1.27 0 180) (size 2 2) (drill 0.8) (layers *.Cu *.Mask)
-      (net 34 "Net-(R1-Pad2)"))
     (pad 1 thru_hole rect (at -3.81 0 180) (size 2 2) (drill 0.8) (layers *.Cu *.Mask)
       (net 2 GND))
@@
   )
   (gr_arc (start 128.27 36.83) (end 132.08 36.83) (angle -90) (layer Edge.Cuts) (width 0.05))
-  (gr_text "ANEMOMETER BOARD\nV1.0" (at 87.63 57.15 90) (layer B.Cu)
+  (gr_text "ANEMOMETER BOARD\nV1.1" (at 87.63 57.15 90) (layer B.Cu)
     (effects (font (size 2.5 2.5) (thickness 0.6)) (justify mirror))
   )
@@
   (segment (start 110.49 58.42) (end 110.49 57.15) (width 1) (layer B.Cu) (net 33))
   (segment (start 110.49 66.04) (end 110.49 58.42) (width 1) (layer B.Cu) (net 33))
-  (segment (start 81.28 91.44) (end 81.28 93.98) (width 1) (layer B.Cu) (net 34))
+  (segment (start 81.28 91.44) (end 81.28 93.98) (width 1) (layer B.Cu) (net 35))
   (segment (start 96.52 92.71) (end 92.71 96.52) (width 1) (layer B.Cu) (net 35))
-  (segment (start 92.71 96.52) (end 77.47 96.52) (width 1) (layer B.Cu) (net 35))
-  (segment (start 76.2 95.25) (end 76.2 93.98) (width 1) (layer B.Cu) (net 35))
-  (segment (start 77.47 96.52) (end 76.2 95.25) (width 1) (layer B.Cu) (net 35))
-  (segment (start 76.2 91.44) (end 76.2 93.98) (width 1) (layer B.Cu) (net 35))
+  (segment (start 76.2 91.44) (end 76.2 93.98) (width 1) (layer B.Cu) (net 34))
+  (segment (start 81.28 95.25) (end 81.28 93.98) (width 1) (layer B.Cu) (net 35))
+  (segment (start 82.55 96.52) (end 81.28 95.25) (width 1) (layer B.Cu) (net 35))
+  (segment (start 92.71 96.52) (end 82.55 96.52) (width 1) (layer B.Cu) (net 35))
   (segment (start 87.63 92.71) (end 86.36 91.44) (width 1) (layer B.Cu) (net 36))
   (segment (start 91.44 92.71) (end 87.63 92.71) (width 1) (layer B.Cu) (net 36))
